File: hw/sch_pcb/REL1SW01.kicad_sch (KiCad schematic)
At the start: 22 parts, among them J1 HEADER_2x02_PARALLEL, J2 HEADER_2x02_PARALLEL, J3 HEADER_2x06_PARALLEL, J4 HEADER_2x06_PARALLEL, J5 HEADER_2x04_PARALLEL, M1 SROUB3M, M2 SROUB3M, M3 SROUB3M, M4 SROUB3M, T1 IRLML6244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

Commit message: update template
Other:
- company: (none) -> www.mlab.cz
- title: (none) -> REL1SW01B
Changed lines of the file:
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@@
 (kicad_sch (version 20230121) (generator eeschema)
   (paper "A4")
+  (title_block
+    (title "REL1SW01B")
+    (date "2024-06-03")
+    (rev "01B")
+    (company "www.mlab.cz")
+    (comment 1 "roman-dvorak <romandvorak@mlab.cz>")
+  )
   (junction (at 168.91 138.43) (diameter 0) (color 0 0 0 0)
   )

Commit message: layout improvements
Other:
- moved on the sheet: C1, C2, D1, D2, D3, D4, J1, J2, J3, J4, J5, M1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
