File: hw/sch_pcb/REL1SW01.kicad_sch (KiCad schematic)
At the start: 22 parts, among them J1 HEADER_2x02_PARALLEL, J2 HEADER_2x02_PARALLEL, J3 HEADER_2x06_PARALLEL, J4 HEADER_2x06_PARALLEL, J5 HEADER_2x04_PARALLEL, M1 SROUB3M, M2 SROUB3M, M3 SROUB3M, M4 SROUB3M, T1 IRLML6244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

Commit message: add ust id
Parts:
- C1: UST_ID (none) -> 60d580ff1287500165f8595a
- C2: UST_ID (none) -> 5c70984712875079b91f8b4c
- D1, D2, D3, D4: UST_ID (none) -> 5c70984512875079b91f88bd
- J1, J2, J3, J4, J5, M1, M2, M3, M4: now left out of the parts list
- R1, R2: UST_ID (none) -> 5c70984512875079b91f8977
- R3, R4: UST_ID (none) -> 639ed3d540d28a66c9e88a9e
- T1, T2: UST_ID (none) -> 5c70984712875079b91f8aef
Changed lines of the file:
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@@
   )
   (symbol (lib_id "MLAB_HEADER:HEADER_2x02_PARALLEL") (at 114.3 64.77 180) (unit 1)
-    (in_bom yes) (on_board yes) (dnp no) (fields_autoplaced)
+    (in_bom no) (on_board yes) (dnp no) (fields_autoplaced)
     (property "Reference" "J1" (at 114.3 59.69 0)
       (effects (font (size 1.524 1.524)))
@@
     (property "Datasheet" "" (at 114.3 66.04 0)
       (effects (font (size 1.524 1.524)))
+    )
+    (property "UST_ID" "" (at 114.3 64.77 0)
+      (effects (font (size 1.27 1.27)) hide)
     )
     (pin "1")
@@
       (effects (font (size 1.27 1.27)) hide)
     )
+    (property "UST_ID" "5c70984712875079b91f8b4c" (at 67.31 27.94 0)
+      (effects (font (size 1.27 1.27)) hide)
+    )
     (pin "2")
     (pin "1")
@@
       (effects (font (size 1.27 1.27)) hide)
     )
+    (property "UST_ID" "5c70984712875079b91f8aef" (at 149.86 97.79 0)
+      (effects (font (size 1.27 1.27)) hide)
+    )
     (pin "1")
     (pin "2")
@@
     )
     (property "Datasheet" "" (at 124.46 154.94 0)
+      (effects (font (size 1.27 1.27)) hide)
+    )
+    (property "UST_ID" "5c70984512875079b91f8977" (at 124.46 154.94 0)
       (effects (font (size 1.27 1.27)) hide)
     )
@@
     )
     (property "Datasheet" "" (at 196.85 101.6 0)
+      (effects (font (size 1.27 1.27)) hide)
+    )
+    (property "UST_ID" "" (at 196.85 101.6 0)
       (effects (font (size 1.27 1.27)) hide)
     )
@@
       (effects (font (size 1.27 1.27)) hide)
     )
+    (property "UST_ID" "639ed3d540d28a66c9e88a9e" (at 134.62 107.95 0)
+      (effects (font (size 1.27 1.27)) hide)
+    )
     (pin "1")
     (pin "2")
@@
   )
   (symbol (lib_id "MLAB_MECHANICAL:HOLE") (at 267.97 40.64 180) (unit 1)
-    (in_bom yes) (on_board yes) (dnp no)
+    (in_bom no) (on_board yes) (dnp no)
     (property "Reference" "M3" (at 270.51 43.18 0)
       (effects (font (size 1.778 1.5113)) (justify left bottom))
@@
     (property "Datasheet" "" (at 267.97 40.64 0)
       (effects (font (size 1.524 1.524)))
+    )
+    (property "UST_ID" "" (at 267.97 40.64 0)
+      (effects (font (size 1.27 1.27)) hide)
     )
     (pin "1")
@@
       (effects (font (size 1.27 1.27)) hide)
     )
+    (property "UST_ID" "5c70984512875079b91f88bd" (at 149.86 140.97 0)
+      (effects (font (size 1.27 1.27)) hide)
+    )
     (pin "1")
     (pin "2")
@@
   )
   (symbol (lib_id "MLAB_HEADER:HEADER_2x02_PARALLEL") (at 147.32 64.77 0) (unit 1)
-    (in_bom yes) (on_board yes) (dnp no) (fields_autoplaced)
+    (in_bom no) (on_board yes) (dnp no) (fields_autoplaced)
     (property "Reference" "J2" (at 151.13 64.77 0)
       (effects (font (size 1.524 1.524)) (justify left))
@@
       (effects (font (size 1.524 1.524)))
     )
+    (property "UST_ID" "" (at 147.32 64.77 0)
+      (effects (font (size 1.27 1.27)) hide)
+    )
     (pin "1")
     (pin "2")
@@
       (effects (font (size 1.27 1.27)) hide)
     )
+    (property "UST_ID" "5c70984512875079b91f88bd" (at 149.86 86.36 0)
+      (effects (font (size 1.27 1.27)) hide)
+    )
     (pin "2")
     (pin "1")
@@
       (effects (font (size 1.27 1.27)) hide)
     )
+    (property "UST_ID" "60d580ff1287500165f8595a" (at 60.96 27.94 0)
+      (effects (font (size 1.27 1.27)) hide)
+    )
     (pin "1")
     (pin "2")
@@
     )
     (property "Datasheet" "" (at 134.62 162.56 0)
+      (effects (font (size 1.27 1.27)) hide)
+    )
+    (property "UST_ID" "639ed3d540d28a66c9e88a9e" (at 134.62 162.56 0)
       (effects (font (size 1.27 1.27)) hide)
     )
@@
       (effects (font (size 1.27 1.27)) hide)
     )
+    (property "UST_ID" "5c70984512875079b91f88bd" (at 142.24 107.95 0)
+      (effects (font (size 1.27 1.27)) hide)
+    )
     (pin "1")
     (pin "2")
@@
       (effects (font (size 1.27 1.27)) hide)
     )
+    (property "UST_ID" "5c70984512875079b91f8977" (at 124.46 100.33 0)
+      (effects (font (size 1.27 1.27)) hide)
+    )
     (pin "1")
     (pin "2")
@@
       (effects (font (size 1.27 1.27)) hide)
     )
+    (property "UST_ID" "5c70984712875079b91f8aef" (at 149.86 152.4 0)
+      (effects (font (size 1.27 1.27)) hide)
+    )
     (pin "1")
     (pin "2")
@@
   )
   (symbol (lib_id "MLAB_MECHANICAL:HOLE") (at 267.97 48.26 180) (unit 1)
-    (in_bom yes) (on_board yes) (dnp no)
+    (in_bom no) (on_board yes) (dnp no)
     (property "Reference" "M4" (at 270.51 50.8 0)
       (effects (font (size 1.778 1.5113)) (justify left bottom))
@@
       (effects (font (size 1.524 1.524)))
     )
+    (property "UST_ID" "" (at 267.97 48.26 0)
+      (effects (font (size 1.27 1.27)) hide)
+    )
     (pin "1")
     (instances
@@
   )
   (symbol (lib_id "MLAB_MECHANICAL:HOLE") (at 267.97 25.4 180) (unit 1)
-    (in_bom yes) (on_board yes) (dnp no)
+    (in_bom no) (on_board yes) (dnp no)
     (property "Reference" "M1" (at 270.51 27.94 0)
       (effects (font (size 1.778 1.5113)) (justify left bottom))
@@
       (effects (font (size 1.524 1.524)))
     )
+    (property "UST_ID" "" (at 267.97 25.4 0)
+      (effects (font (size 1.27 1.27)) hide)
+    )
     (pin "1")
     (instances
@@
   )
   (symbol (lib_id "MLAB_HEADER:HEADER_2x06_PARALLEL") (at 195.58 86.36 90) (unit 1)
-    (in_bom yes) (on_board yes) (dnp no) (fields_autoplaced)
+    (in_bom no) (on_board yes) (dnp no) (fields_autoplaced)
     (property "Reference" "J3" (at 204.47 86.36 90)
       (effects (font (size 1.524 1.524)) (justify right))
@@
     (property "Datasheet" "" (at 189.23 86.36 0)
       (effects (font (size 1.524 1.524)))
+    )
+    (property "UST_ID" "" (at 195.58 86.36 0)
+      (effects (font (size 1.27 1.27)) hide)
     )
     (pin "11")
@@
   )
   (symbol (lib_id "MLAB_HEADER:HEADER_2x06_PARALLEL") (at 195.58 116.84 270) (unit 1)
-    (in_bom yes) (on_board yes) (dnp no) (fields_autoplaced)
+    (in_bom no) (on_board yes) (dnp no) (fields_autoplaced)
     (property "Reference" "J4" (at 204.47 116.84 90)
       (effects (font (size 1.524 1.524)) (justify left))
@@
     (property "Datasheet" "" (at 201.93 116.84 0)
       (effects (font (size 1.524 1.524)))
+    )
+    (property "UST_ID" "" (at 195.58 116.84 0)
+      (effects (font (size 1.27 1.27)) hide)
     )
     (pin "11")
@@
       (effects (font (size 1.27 1.27)) hide)
     )
+    (property "UST_ID" "5c70984512875079b91f88bd" (at 142.24 162.56 0)
+      (effects (font (size 1.27 1.27)) hide)
+    )
     (pin "2")
     (pin "1")
@@
   )
   (symbol (lib_id "MLAB_HEADER:HEADER_2x04_PARALLEL") (at 39.37 30.48 0) (unit 1)
-    (in_bom yes) (on_board yes) (dnp no) (fields_autoplaced)
+    (in_bom no) (on_board yes) (dnp no) (fields_autoplaced)
     (property "Reference" "J5" (at 43.18 30.48 0)
       (effects (font (size 1.524 1.524)) (justify left))
@@
     (property "Datasheet" "" (at 39.37 26.67 0)
       (effects (font (size 1.524 1.524)))
+    )
+    (property "UST_ID" "" (at 39.37 30.48 0)
+      (effects (font (size 1.27 1.27)) hide)
     )
     (pin "6")
@@
   )
   (symbol (lib_id "MLAB_MECHANICAL:HOLE") (at 267.97 33.02 180) (unit 1)
-    (in_bom yes) (on_board yes) (dnp no)
+    (in_bom no) (on_board yes) (dnp no)
     (property "Reference" "M2" (at 270.51 35.56 0)
       (effects (font (size 1.778 1.5113)) (justify left bottom))
@@
       (effects (font (size 1.524 1.524)))
     )
-    (pin "1")
+    (property "UST_ID" "" (at 267.97 33.02 0)
+      (effects (font (size 1.27 1.27)) hide)
+    )
+    (pin "1")
