File: hw/sch_pcb/REL1SW01.kicad_pcb (KiCad board)
At the start: 2 copper layers, 30 x 40.1 mm, 22 parts, among them J1 HEADER_2x02_PARALLEL, J2 HEADER_2x02_PARALLEL, J3 HEADER_2x06_PARALLEL, J4 HEADER_2x06_PARALLEL, J5 HEADER_2x04_PARALLEL, M1 SROUB3M, M2 SROUB3M, M3 SROUB3M, M4 SROUB3M, T1 IRLML6244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

Commit message: update template
Parts:
- moved J2 0.20 mm to (158.8, 97.4)
Changed lines of the file:
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@@
   )
   (paper "A4")
+  (title_block
+    (title "REL1SW01B")
+    (date "2024-06-03")
+    (rev "01B")
+    (company "www.mlab.cz")
+    (comment 1 "roman-dvorak <romandvorak@mlab.cz>")
+  )
   (layers
     (0 "F.Cu" signal)
@@
   )
   (footprint "Mlab_Pin_Headers:Straight_2x02" (layer "F.Cu")
-    (at 158.609999 97.43)
+    (at 158.809999 97.43)
     (descr "pin header straight 2x02")
     (tags "pin header straight 2x02")
@@
     )
   )
-  (gr_line (start 147.879999 100) (end 149.679999 100)
-    (stroke (width 0.2) (type default)) (layer "F.SilkS"))
-  (gr_line (start 147.479999 98.5) (end 147.479999 100.2)
-    (stroke (width 0.2) (type default)) (layer "F.SilkS"))
-  (gr_line (start 149.179999 98.7) (end 151.279999 98.7)
+  (gr_line (start 147.879999 100.2) (end 149.679999 100.2)
+    (stroke (width 0.2) (type default)) (layer "F.SilkS"))
+  (gr_line (start 147.479999 98.7) (end 147.479999 100.4)
+    (stroke (width 0.2) (type default)) (layer "F.SilkS"))
+  (gr_line (start 149.179999 98.9) (end 151.279999 98.9)
     (stroke (width 0.2) (type default)) (layer "F.SilkS"))
   (gr_line (start 149.579999 97.7) (end 149.779999 97.7)
     (stroke (width 0.2) (type default)) (layer "F.SilkS"))
-  (gr_line (start 149.679999 100) (end 149.679999 100.6)
+  (gr_line (start 149.679999 100.2) (end 149.679999 100.8)
     (stroke (width 0.2) (type default)) (layer "F.SilkS"))
   (gr_line (start 147.479999 96.3) (end 144.479999 96.3)
@@
   (gr_line (start 147.879999 96.8) (end 147.879999 96.4)
     (stroke (width 0.2) (type default)) (layer "F.SilkS"))
-  (gr_line (start 147.879999 98.7) (end 149.179999 98.7)
+  (gr_line (start 147.879999 98.9) (end 149.179999 98.9)
     (stroke (width 0.2) (type default)) (layer "F.SilkS"))
   (gr_line (start 147.879999 95.2) (end 149.179999 95.2)
     (stroke (width 0.2) (type default)) (layer "F.SilkS"))
-  (gr_line (start 147.879999 98.4) (end 147.879999 98.8)
+  (gr_line (start 147.879999 98.6) (end 147.879999 99)
     (stroke (width 0.2) (type default)) (layer "F.SilkS"))
   (gr_line (start 149.479999 97.4) (end 149.879999 97.4)
     (stroke (width 0.2) (type default)) (layer "F.SilkS"))
-  (gr_circle (center 147.976433 99.4) (end 149.376433 99.5)
+  (gr_circle (center 147.976433 99.6) (end 149.376433 99.7)
     (stroke (width 0.2) (type default)) (fill none) (layer "F.SilkS"))
-  (gr_line (start 147.879999 99.6) (end 147.879999 99.1)
+  (gr_line (start 147.879999 99.8) (end 147.879999 99.3)
     (stroke (width 0.2) (type default)) (layer "F.SilkS"))
   (gr_line (start 149.279999 97.1) (end 150.079999 97.1)
     (stroke (width 0.2) (type default)) (layer "F.SilkS"))
-  (gr_line (start 149.479999 100.9) (end 149.879999 100.9)
+  (gr_line (start 149.479999 101.1) (end 149.879999 101.1)
     (stroke (width 0.2) (type default)) (layer "F.SilkS"))
   (gr_line (start 147.879999 94.9) (end 147.879999 95.3)
@@
   (gr_line (start 149.679999 96.5) (end 149.679999 97.1)
     (stroke (width 0.2) (type default)) (layer "F.SilkS"))
-  (gr_line (start 147.879999 100.3) (end 147.879999 99.9)
-    (stroke (width 0.2) (type default)) (layer "F.SilkS"))
-  (gr_line (start 147.479999 99.8) (end 144.479999 99.8)
+  (gr_line (start 147.879999 100.5) (end 147.879999 100.1)
+    (stroke (width 0.2) (type default)) (layer "F.SilkS"))
+  (gr_line (start 147.479999 100) (end 144.479999 100)
     (stroke (width 0.2) (type default)) (layer "F.SilkS"))
   (gr_circle (center 147.976433 95.9) (end 149.376433 96)
@@
   (gr_line (start 147.879999 96.1) (end 147.879999 95.6)
     (stroke (width 0.2) (type default)) (layer "F.SilkS"))
-  (gr_line (start 149.279999 100.6) (end 150.079999 100.6)
+  (gr_line (start 149.279999 100.8) (end 150.079999 100.8)
     (stroke (width 0.2) (type default)) (layer "F.SilkS"))
   (gr_line (start 149.179999 95.2) (end 151.279999 95.2)
     (stroke (width 0.2) (type default)) (layer "F.SilkS"))
-  (gr_line (start 149.579999 101.2) (end 149.779999 101.2)
+  (gr_line (start 149.579999 101.4) (end 149.779999 101.4)
     (stroke (width 0.2) (type default)) (layer "F.SilkS"))
   (gr_rect (start 133.513999 84.934) (end 163.486 125.066)
@@
     (effects (font (size 1.2 1.2) (thickness 0.2) bold) (justify left bottom))
   )
-  (gr_text "OUT2" (at 151.279999 99.5) (layer "F.SilkS")
+  (gr_text "OUT2" (at 151.479999 99.5) (layer "F.SilkS")
     (effects (font (size 1.2 1.2) (thickness 0.2) bold) (justify left bottom))
   )
@@
     (effects (font (size 1.2 1.2) (thickness 0.2) bold) (justify left bottom))
   )
-  (gr_text "OUT1" (at 151.279999 96.8) (layer "F.SilkS")
-    (effects (font (size 1.2 1.2) (thickness 0.2) bold) (justify left bottom))
-  )
-  (gr_text "POWER" (at 148.176433 93.7) (layer "F.SilkS")
+  (gr_text "OUT1" (at 151.479999 96.8) (layer "F.SilkS")
+    (effects (font (size 1.2 1.2) (thickness 0.2) bold) (justify left bottom))
+  )
+  (gr_text "POWER" (at 148.176433 93.5) (layer "F.SilkS")
     (effects (font (size 1.8 1.8) (thickness 0.2)) (justify bottom))
   )
@@
     (connect_pads (clearance 0.000001))
     (min_thickness 0.2032) (filled_areas_thickness no)
-    (fill (thermal_gap 0.25) (thermal_bridge_width 0.4564))
+    (fill yes (thermal_gap 0.25) (thermal_bridge_width 0.4564))
     (polygon
       (pts

Commit message: layout improvements
Parts:
- moved X1 1.00 mm to (144.8, 107.3)
Routing:
- net +VCC: track 78.5 -> 79.3 mm
- net /OUT1: track 9.11 -> 8.61 mm
Changed lines of the file:
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@@
   (net 18 "Net-(D2-K)")
   (footprint "Relay_THT:Relay_DPDT_FRT5" (layer "F.Cu")
-    (at 144.654999 108.3)
+    (at 144.754999 107.3)
     (descr "IM Signal Relay DPDT FRT5 narrow footprint")
     (tags "Relay DPDT IM-relay FRT5")
@@
   (segment (start 149.4 102.019999) (end 149.4 87.33) (width 0.8) (layer "F.Cu") (net 1))
   (segment (start 149.4 87.3) (end 149.4 90.820001) (width 0.8) (layer "B.Cu") (net 1))
-  (segment (start 150.979999 92.1) (end 150.979999 93.1) (width 0.8) (layer "B.Cu") (net 1))
-  (segment (start 160.479999 101.5) (end 154.279999 101.5) (width 0.8) (layer "B.Cu") (net 1))
-  (segment (start 162.079999 95.2) (end 162.079999 99.9) (width 0.8) (layer "B.Cu") (net 1))
-  (segment (start 150.979999 93.1) (end 152.039999 94.16) (width 0.8) (layer "B.Cu") (net 1))
-  (segment (start 149.4 90.820001) (end 149.379999 90.840002) (width 0.8) (layer "B.Cu") (net 1))
+  (segment (start 152.439999 94.16) (end 161.139999 94.16) (width 0.8) (layer "B.Cu") (net 1))
+  (segment (start 162.079999 99.9) (end 160.479999 101.5) (width 0.8) (layer "B.Cu") (net 1))
+  (segment (start 161.139999 94.16) (end 162.079999 95.1) (width 0.8) (layer "B.Cu") (net 1))
+  (segment (start 149.4 89.87) (end 149.4 92.079999) (width 0.8) (layer "B.Cu") (net 1))
+  (segment (start 150.979999 92.7) (end 152.439999 94.16) (width 0.8) (layer "B.Cu") (net 1))
+  (segment (start 146.89 87.3) (end 149.4 87.3) (width 0.8) (layer "B.Cu") (net 1))
+  (segment (start 162.079999 95.1) (end 162.079999 99.9) (width 0.8) (layer "B.Cu") (net 1))
+  (segment (start 149.379999 92.1) (end 150.979999 92.1) (width 0.8) (layer "B.Cu") (net 1))
+  (segment (start 149.4 89.87) (end 146.86 89.87) (width 0.5) (layer "B.Cu") (net 1))
+  (segment (start 149.4 92.079999) (end 149.379999 92.1) (width 0.8) (layer "B.Cu") (net 1))
+  (segment (start 150.979999 92.1) (end 150.979999 92.7) (width 0.8) (layer "B.Cu") (net 1))
   (segment (start 154.279999 101.5) (end 154.179999 101.6) (width 0.8) (layer "B.Cu") (net 1))
-  (segment (start 146.89 87.3) (end 149.4 87.3) (width 0.8) (layer "B.Cu") (net 1))
-  (segment (start 162.079999 99.9) (end 160.479999 101.5) (width 0.8) (layer "B.Cu") (net 1))
-  (segment (start 149.379999 90.840002) (end 149.379999 92.1) (width 0.8) (layer "B.Cu") (net 1))
-  (segment (start 149.4 89.87) (end 146.86 89.87) (width 0.5) (layer "B.Cu") (net 1))
-  (segment (start 161.039999 94.16) (end 162.079999 95.2) (width 0.8) (layer "B.Cu") (net 1))
-  (segment (start 150.979999 92.1) (end 149.379999 92.1) (width 0.5) (layer "B.Cu") (net 1))
-  (segment (start 152.039999 94.16) (end 161.039999 94.16) (width 0.8) (layer "B.Cu") (net 1))
   (segment (start 146.86 87.33) (end 146.89 87.3) (width 0.8) (layer "B.Cu") (net 1))
   (segment (start 154.179999 100.4) (end 154.179999 103.6) (width 0.8) (layer "B.Cu") (net 1))
+  (segment (start 160.479999 101.5) (end 154.279999 101.5) (width 0.8) (layer "B.Cu") (net 1))
   (segment (start 140.979999 98.6) (end 141.854999 99.475) (width 0.5) (layer "B.Cu") (net 3))
   (segment (start 137.364999 98.6) (end 140.979999 98.6) (width 0.5) (layer "B.Cu") (net 3))
-  (segment (start 137.104999 96.06) (end 140.639999 96.06) (width 0.5) (layer "B.Cu") (net 4))
-  (segment (start 140.639999 96.06) (end 143.867499 99.2875) (width 0.5) (layer "B.Cu") (net 4))
-  (segment (start 143.867499 99.2875) (end 143.867499 99.4) (width 0.5) (layer "B.Cu") (net 4))
+  (segment (start 137.104999 96.06) (end 140.739999 96.06) (width 0.5) (layer "B.Cu") (net 4))
+  (segment (start 143.867499 99.1875) (end 143.867499 99.4) (width 0.5) (layer "B.Cu") (net 4))
+  (segment (start 140.739999 96.06) (end 143.867499 99.1875) (width 0.5) (layer "B.Cu") (net 4))
   (segment (start 159.519999 95.8) (end 159.879999 96.16) (width 0.8) (layer "B.Cu") (net 5))
-  (segment (start 150.917499 95.8) (end 159.519999 95.8) (width 0.8) (layer "B.Cu") (net 5))
+  (segment (start 151.417499 95.8) (end 159.519999 95.8) (width 0.8) (layer "B.Cu") (net 5))
   (segment (start 151.379999 99.3) (end 152.279999 98.4) (width 0.8) (layer "B.Cu") (net 6))
   (segment (start 152.279999 98.4) (end 159.579999 98.4) (width 0.8) (layer "B.Cu") (net 6))
@@
   (segment (start 150.779999 103.6) (end 151.379999 103) (width 0.8) (layer "B.Cu") (net 6))
   (segment (start 151.379999 103) (end 151.379999 99.3) (width 0.8) (layer "B.Cu") (net 6))
-  (segment (start 157.099999 104.58) (end 153.379999 108.3) (width 0.8) (layer "B.Cu") (net 7))
-  (segment (start 153.379999 108.3) (end 152.274999 108.3) (width 0.8) (layer "B.Cu") (net 7))
   (segment (start 160.049999 104.58) (end 157.099999 104.58) (width 0.8) (layer "B.Cu") (net 7))
-  (segment (start 153.339999 110.84) (end 152.274999 110.84) (width 0.8) (layer "B.Cu") (net 8))
-  (segment (start 157.059999 107.12) (end 153.339999 110.84) (width 0.8) (layer "B.Cu") (net 8))
+  (segment (start 154.379999 107.3) (end 152.274999 107.3) (width 0.8) (layer "B.Cu") (net 7))
+  (segment (start 157.099999 104.58) (end 154.379999 107.3) (width 0.8) (layer "B.Cu") (net 7))
   (segment (start 160.049999 107.12) (end 157.059999 107.12) (width 0.8) (layer "B.Cu") (net 8))
+  (segment (start 157.059999 107.12) (end 154.339999 109.84) (width 0.8) (layer "B.Cu") (net 8))
+  (segment (start 154.339999 109.84) (end 152.274999 109.84) (width 0.8) (layer "B.Cu") (net 8))
   (segment (start 160.049999 109.66) (end 157.019999 109.66) (width 0.8) (layer "B.Cu") (net 9))
-  (segment (start 157.019999 109.66) (end 153.299999 113.38) (width 0.8) (layer "B.Cu") (net 9))
-  (segment (start 153.299999 113.38) (end 152.274999 113.38) (width 0.8) (layer "B.Cu") (net 9))
-  (segment (start 153.267499 115.92) (end 152.274999 115.92) (width 0.8) (layer "B.Cu") (net 10))
-  (segment (start 156.987499 112.2) (end 153.267499 115.92) (width 0.8) (layer "B.Cu") (net 10))
+  (segment (start 154.299999 112.38) (end 152.274999 112.38) (width 0.8) (layer "B.Cu") (net 9))
+  (segment (start 157.019999 109.66) (end 154.299999 112.38) (width 0.8) (layer "B.Cu") (net 9))
+  (segment (start 156.987499 112.2) (end 154.267499 114.92) (width 0.8) (layer "B.Cu") (net 10))
+  (segment (start 154.267499 114.92) (end 152.274999 114.92) (width 0.8) (layer "B.Cu") (net 10))
   (segment (start 160.049999 112.2) (end 156.987499 112.2) (width 0.8) (layer "B.Cu") (net 10))
-  (segment (start 157.039999 114.74) (end 153.319999 118.46) (width 0.8) (layer "B.Cu") (net 11))
+  (segment (start 154.319999 117.46) (end 152.274999 117.46) (width 0.8) (layer "B.Cu") (net 11))
   (segment (start 160.049999 114.74) (end 157.039999 114.74) (width 0.8) (layer "B.Cu") (net 11))
-  (segment (start 153.319999 118.46) (end 152.274999 118.46) (width 0.8) (layer "B.Cu") (net 11))
-  (segment (start 140.219999 114.74) (end 143.939999 118.46) (width 0.8) (layer "B.Cu") (net 12))
+  (segment (start 157.039999 114.74) (end 154.319999 117.46) (width 0.8) (layer "B.Cu") (net 11))
+  (segment (start 140.219999 114.74) (end 142.939999 117.46) (width 0.8) (layer "B.Cu") (net 12))
+  (segment (start 142.939999 117.46) (end 144.654999 117.46) (width 0.8) (layer "B.Cu") (net 12))
   (segment (start 137.209999 114.74) (end 140.219999 114.74) (width 0.8) (layer "B.Cu") (net 12))
-  (segment (start 143.939999 118.46) (end 144.654999 118.46) (width 0.8) (layer "B.Cu") (net 12))
-  (segment (start 143.799999 115.92) (end 144.654999 115.92) (width 0.8) (layer "B.Cu") (net 13))
-  (segment (start 140.079999 112.2) (end 143.799999 115.92) (width 0.8) (layer "B.Cu") (net 13))
+  (segment (start 142.799999 114.92) (end 144.654999 114.92) (width 0.8) (layer "B.Cu") (net 13))
   (segment (start 137.209999 112.2) (end 140.079999 112.2) (width 0.8) (layer "B.Cu") (net 13))
-  (segment (start 143.957499 113.38) (end 144.654999 113.38) (width 0.8) (layer "B.Cu") (net 14))
+  (segment (start 140.079999 112.2) (end 142.799999 114.92) (width 0.8) (layer "B.Cu") (net 13))
+  (segment (start 142.957499 112.38) (end 144.654999 112.38) (width 0.8) (layer "B.Cu") (net 14))
+  (segment (start 140.237499 109.66) (end 142.957499 112.38) (width 0.8) (layer "B.Cu") (net 14))
   (segment (start 137.209999 109.66) (end 140.237499 109.66) (width 0.8) (layer "B.Cu") (net 14))
-  (segment (start 140.237499 109.66) (end 143.957499 113.38) (width 0.8) (layer "B.Cu") (net 14))
+  (segment (start 143.037499 109.84) (end 144.654999 109.84) (width 0.8) (layer "B.Cu") (net 15))
+  (segment (start 140.317499 107.12) (end 143.037499 109.84) (width 0.8) (layer "B.Cu") (net 15))
   (segment (start 137.209999 107.12) (end 140.317499 107.12) (width 0.8) (layer "B.Cu") (net 15))
-  (segment (start 144.037499 110.84) (end 144.654999 110.84) (width 0.8) (layer "B.Cu") (net 15))
-  (segment (start 140.317499 107.12) (end 144.037499 110.84) (width 0.8) (layer "B.Cu") (net 15))
+  (segment (start 140.259999 104.58) (end 142.979999 107.3) (width 0.8) (layer "B.Cu") (net 16))
+  (segment (start 142.979999 107.3) (end 144.654999 107.3) (width 0.8) (layer "B.Cu") (net 16))
   (segment (start 137.209999 104.58) (end 140.259999 104.58) (width 0.8) (layer "B.Cu") (net 16))
-  (segment (start 140.259999 104.58) (end 143.979999 108.3) (width 0.8) (layer "B.Cu") (net 16))
-  (segment (start 143.979999 108.3) (end 144.654999 108.3) (width 0.8) (layer "B.Cu") (net 16))
   (segment (start 144.767499 96.7125) (end 144.679999 96.8) (width 0.5) (layer "B.Cu") (net 17))
   (segment (start 149.042499 96.75) (end 149.004999 96.7125) (width 0.5) (layer "B.Cu") (net 17))
